Commit message: Updated submission for checkpoint7 task2

File: xacro/drive_wheel.xacro (robot description, xacro)
@@ -4,7 +4,7 @@
 <link name="base_${side}_wheel_link">
   <inertial>
-    <mass value="3"/>
-    <inertia ixx="0.0014" iyy="0.0014" izz="0.0025" ixy="0" ixz="0" iyz="0"/>
-  </inertial>
+    <mass value="2"/>
+    <inertia ixx="0.00013" iyy="0.00013" izz="0.00021" ixy="0" ixz="0" iyz="0"/>
+</inertial>
   <visual>
     <geometry>
