Commit message: Updated urdf file for task1

File: urdf/barista_robot_model.urdf (robot description, URDF)
Before this commit: robot barista_robot, 17 links, 16 joints
Links:
- link base_left_wheel_link: mass 3 -> 2
- link base_right_wheel_link: mass 3 -> 2
Joints:
- joint left_wheel_joint: origin xyz=0 -0.155 0.0352 rpy=-1.57 0 0 -> xyz=0 0.155 0.0352 rpy=-1.57 0 0
- joint right_wheel_joint: origin xyz=0 0.155 0.0352 rpy=-1.57 0 0 -> xyz=0 -0.155 0.0352 rpy=-1.57 0 0

Commit message: Update barista_robot_model.urdf

File: urdf/barista_robot_model.urdf (robot description, URDF)
Before this commit: robot barista_robot, 17 links, 16 joints
Links:
- link laser_scan_link: geometry collision box size=0.1 0.1 0.1; visual mesh filename=package://barista_robot_description/models/meshes/hokuyo_ur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 scale=1 1 1
Joints:
- joint laser_joint: origin xyz=0 0 0 rpy=0 0 0 -> xyz=0.14 0 0.2 rpy=0 0 0
- joint laser_joint_frame: origin xyz=0.14 0 0.2 rpy=0 0 0 -> xyz=0 0 0.05 rpy=0 0 0
